Commit message: 🦊Foxglove configs added

File: description/viam_rover_description.urdf (robot description, URDF)
Before this commit: robot viam_rover, 5 links, 4 joints
Links:
- link base_link: geometry visual box size=0.21 0.31 0.075
- link left_wheel: geometry visual cylinder length=0.03 radius=0.052
- link right_wheel: geometry visual cylinder length=0.03 radius=0.052
Joints:
- joint default_cam_joint: origin xyz=0.2 0.0 0.1 rpy=1.57 3.14 1.57 -> xyz=0.1 0.0 0.11 rpy=1.57 3.14 1.57
- joint left_wheel_joint: origin xyz=0.0 -0.13 -0.02 rpy=0 0 0 -> xyz=0.0 -0.16 0.03 rpy=0 0 0
- joint right_wheel_joint: origin xyz=0.0 0.13 -0.02 rpy=0 0 0 -> xyz=0.0 0.16 0.03 rpy=0 0 0
- joint scan_joint: origin xyz=0.2 0.0 0.1 rpy=0.0 0.0 0.0 -> xyz=0.1 0.0 0.11 rpy=0.0 0.0 0.0
